File: Picon_kicad/Picon_kicad.sch (KiCad schematic (older format))
At the start: 43 parts, among them U1 Pico

Commit message: v0.2 | Rudimentary PCB layout
Parts:
- R1, R10, R11, R12, R13, R14, R15, R16, R17, R2, R3, R4, R5, R6, R7, R8, R9: footprint Resistor_THT:R_Axial_DIN0207_L6.3mm_D2.5mm_P7.62mm_Horizontal -> Resistor_SMD:R_0603_1608Metric
- U1: footprint RPi_Pico:RPi_Pico_SMD_TH -> MCU_RaspberryPi_and_Boards:RPi_Pico_SMD_TH
- USBC1: footprint Type-C:HRO-TYPE-C-31-M-12-HandSoldering -> Type-C:HRO-TYPE-C-31-M-12-Assembly
Changed lines of the file:
@@
 F 0 "U1" V 2146 4356 50  0000 R CNN
 F 1 "Pico" V 2055 4356 50  0000 R CNN
-F 2 "RPi_Pico:RPi_Pico_SMD_TH" V 2100 5550 50  0001 C CNN
+F 2 "MCU_RaspberryPi_and_Boards:RPi_Pico_SMD_TH" V 2100 5550 50  0001 C CNN
 F 3 "" H 2100 5550 50  0001 C CNN
 	1    2100 5550
@@
 F 0 "USBC1" V 1980 2088 60  0000 L CNN
 F 1 "HRO-TYPE-C-31-M-12" V 2086 2088 60  0000 L CNN
-F 2 "Type-C:HRO-TYPE-C-31-M-12-HandSoldering" H 2200 1450 60  0001 C CNN
+F 2 "Type-C:HRO-TYPE-C-31-M-12-Assembly" H 2200 1450 60  0001 C CNN
 F 3 "" H 2200 1450 60  0001 C CNN
 F 4 "C165948" V 2200 1450 50  0001 C CNN "LCSC"
@@
 F 0 "R16" H 1909 1946 50  0000 L CNN
 F 1 "5K1" H 1909 1855 50  0000 L CNN
-F 2 "Resistor_THT:R_Axial_DIN0207_L6.3mm_D2.5mm_P7.62mm_Horizontal" H 1850 1900 50  0001 C CNN
+F 2 "Resistor_SMD:R_0603_1608Metric" H 1850 1900 50  0001 C CNN
 F 3 "~" H 1850 1900 50  0001 C CNN
 F 4 "C23186" H 1850 1900 50  0001 C CNN "LCSC"
@@
 F 0 "R17" H 2509 1946 50  0000 L CNN
 F 1 "5K1" H 2509 1855 50  0000 L CNN
-F 2 "Resistor_THT:R_Axial_DIN0207_L6.3mm_D2.5mm_P7.62mm_Horizontal" H 2450 1900 50  0001 C CNN
+F 2 "Resistor_SMD:R_0603_1608Metric" H 2450 1900 50  0001 C CNN
 F 3 "~" H 2450 1900 50  0001 C CNN
 F 4 "C23186" H 2450 1900 50  0001 C CNN "LCSC"
@@
 F 0 "R1" V 4854 2050 50  0000 C CNN
 F 1 "120R" V 4945 2050 50  0000 C CNN
-F 2 "Resistor_THT:R_Axial_DIN0207_L6.3mm_D2.5mm_P7.62mm_Horizontal" H 5050 2050 50  0001 C CNN
+F 2 "Resistor_SMD:R_0603_1608Metric" H 5050 2050 50  0001 C CNN
 F 3 "~" H 5050 2050 50  0001 C CNN
 F 4 "C22787" V 5050 2050 50  0001 C CNN "LCSC"
@@
 F 0 "R2" V 5854 2050 50  0000 C CNN
 F 1 "120R" V 5945 2050 50  0000 C CNN
-F 2 "Resistor_THT:R_Axial_DIN0207_L6.3mm_D2.5mm_P7.62mm_Horizontal" H 6050 2050 50  0001 C CNN
+F 2 "Resistor_SMD:R_0603_1608Metric" H 6050 2050 50  0001 C CNN
 F 3 "~" H 6050 2050 50  0001 C CNN
 F 4 "C22787" V 6050 2050 50  0001 C CNN "LCSC"
@@
 F 0 "R3" V 6854 2050 50  0000 C CNN
 F 1 "120R" V 6945 2050 50  0000 C CNN
-F 2 "Resistor_THT:R_Axial_DIN0207_L6.3mm_D2.5mm_P7.62mm_Horizontal" H 7050 2050 50  0001 C CNN
+F 2 "Resistor_SMD:R_0603_1608Metric" H 7050 2050 50  0001 C CNN
 F 3 "~" H 7050 2050 50  0001 C CNN
 F 4 "C22787" V 7050 2050 50  0001 C CNN "LCSC"
@@
 F 0 "R4" V 7854 2050 50  0000 C CNN
 F 1 "120R" V 7945 2050 50  0000 C CNN
-F 2 "Resistor_THT:R_Axial_DIN0207_L6.3mm_D2.5mm_P7.62mm_Horizontal" H 8050 2050 50  0001 C CNN
+F 2 "Resistor_SMD:R_0603_1608Metric" H 8050 2050 50  0001 C CNN
 F 3 "~" H 8050 2050 50  0001 C CNN
 F 4 "C22787" V 8050 2050 50  0001 C CNN "LCSC"
@@
 F 0 "R5" V 4854 3050 50  0000 C CNN
 F 1 "120R" V 4945 3050 50  0000 C CNN
-F 2 "Resistor_THT:R_Axial_DIN0207_L6.3mm_D2.5mm_P7.62mm_Horizontal" H 5050 3050 50  0001 C CNN
+F 2 "Resistor_SMD:R_0603_1608Metric" H 5050 3050 50  0001 C CNN
 F 3 "~" H 5050 3050 50  0001 C CNN
 F 4 "C22787" V 5050 3050 50  0001 C CNN "LCSC"
@@
 F 0 "R6" V 5854 3050 50  0000 C CNN
 F 1 "120R" V 5945 3050 50  0000 C CNN
-F 2 "Resistor_THT:R_Axial_DIN0207_L6.3mm_D2.5mm_P7.62mm_Horizontal" H 6050 3050 50  0001 C CNN
+F 2 "Resistor_SMD:R_0603_1608Metric" H 6050 3050 50  0001 C CNN
 F 3 "~" H 6050 3050 50  0001 C CNN
 F 4 "C22787" V 6050 3050 50  0001 C CNN "LCSC"
@@
 F 0 "R7" V 6854 3050 50  0000 C CNN
 F 1 "120R" V 6945 3050 50  0000 C CNN
-F 2 "Resistor_THT:R_Axial_DIN0207_L6.3mm_D2.5mm_P7.62mm_Horizontal" H 7050 3050 50  0001 C CNN
+F 2 "Resistor_SMD:R_0603_1608Metric" H 7050 3050 50  0001 C CNN
 F 3 "~" H 7050 3050 50  0001 C CNN
 F 4 "C22787" V 7050 3050 50  0001 C CNN "LCSC"
@@
 F 0 "R8" V 7854 3050 50  0000 C CNN
 F 1 "120R" V 7945 3050 50  0000 C CNN
-F 2 "Resistor_THT:R_Axial_DIN0207_L6.3mm_D2.5mm_P7.62mm_Horizontal" H 8050 3050 50  0001 C CNN
+F 2 "Resistor_SMD:R_0603_1608Metric" H 8050 3050 50  0001 C CNN
 F 3 "~" H 8050 3050 50  0001 C CNN
 F 4 "C22787" V 8050 3050 50  0001 C CNN "LCSC"
@@
 F 0 "R9" V 8854 3050 50  0000 C CNN
 F 1 "120R" V 8945 3050 50  0000 C CNN
-F 2 "Resistor_THT:R_Axial_DIN0207_L6.3mm_D2.5mm_P7.62mm_Horizontal" H 9050 3050 50  0001 C CNN
+F 2 "Resistor_SMD:R_0603_1608Metric" H 9050 3050 50  0001 C CNN
 F 3 "~" H 9050 3050 50  0001 C CNN
 F 4 "C22787" V 9050 3050 50  0001 C CNN "LCSC"
@@
 F 0 "R10" V 4704 4500 50  0000 C CNN
 F 1 "120R" V 4795 4500 50  0000 C CNN
-F 2 "Resistor_THT:R_Axial_DIN0207_L6.3mm_D2.5mm_P7.62mm_Horizontal" H 4900 4500 50  0001 C CNN
+F 2 "Resistor_SMD:R_0603_1608Metric" H 4900 4500 50  0001 C CNN
 F 3 "~" H 4900 4500 50  0001 C CNN
 F 4 "C22787" V 4900 4500 50  0001 C CNN "LCSC"
@@
 F 0 "R11" V 5704 4500 50  0000 C CNN
 F 1 "120R" V 5795 4500 50  0000 C CNN
-F 2 "Resistor_THT:R_Axial_DIN0207_L6.3mm_D2.5mm_P7.62mm_Horizontal" H 5900 4500 50  0001 C CNN
+F 2 "Resistor_SMD:R_0603_1608Metric" H 5900 4500 50  0001 C CNN
 F 3 "~" H 5900 4500 50  0001 C CNN
 F 4 "C22787" V 5900 4500 50  0001 C CNN "LCSC"
@@
 F 0 "R12" V 4954 5150 50  0000 C CNN
 F 1 "120R" V 5045 5150 50  0000 C CNN
-F 2 "Resistor_THT:R_Axial_DIN0207_L6.3mm_D2.5mm_P7.62mm_Horizontal" H 5150 5150 50  0001 C CNN
+F 2 "Resistor_SMD:R_0603_1608Metric" H 5150 5150 50  0001 C CNN
 F 3 "~" H 5150 5150 50  0001 C CNN
 F 4 "C22787" V 5150 5150 50  0001 C CNN "LCSC"
@@
 F 0 "R13" V 6454 5150 50  0000 C CNN
 F 1 "120R" V 6545 5150 50  0000 C CNN
-F 2 "Resistor_THT:R_Axial_DIN0207_L6.3mm_D2.5mm_P7.62mm_Horizontal" H 6650 5150 50  0001 C CNN
+F 2 "Resistor_SMD:R_0603_1608Metric" H 6650 5150 50  0001 C CNN
 F 3 "~" H 6650 5150 50  0001 C CNN
 F 4 "C22787" V 6650 5150 50  0001 C CNN "LCSC"
@@
 F 0 "R14" V 7954 5150 50  0000 C CNN
 F 1 "120R" V 8045 5150 50  0000 C CNN
-F 2 "Resistor_THT:R_Axial_DIN0207_L6.3mm_D2.5mm_P7.62mm_Horizontal" H 8150 5150 50  0001 C CNN
+F 2 "Resistor_SMD:R_0603_1608Metric" H 8150 5150 50  0001 C CNN
 F 3 "~" H 8150 5150 50  0001 C CNN
 F 4 "C22787" V 8150 5150 50  0001 C CNN "LCSC"
@@
 F 0 "R15" V 9454 5150 50  0000 C CNN
 F 1 "120R" V 9545 5150 50  0000 C CNN
-F 2 "Resistor_THT:R_Axial_DIN0207_L6.3mm_D2.5mm_P7.62mm_Horizontal" H 9650 5150 50  0001 C CNN
+F 2 "Resistor_SMD:R_0603_1608Metric" H 9650 5150 50  0001 C CNN
 F 3 "~" H 9650 5150 50  0001 C CNN
 F 4 "C22787" V 9650 5150 50  0001 C CNN "LCSC"
